File: Microwave/pcb/microwave-coil/microwave-coil.kicad_pcb (KiCad board)
At the start: 2 copper layers, 50.8 x 25.4 mm, 1 part

Commit message: save new version
Parts:
- added REF**: signal, custom:open-mask, F.Cu at (75.3, 100.2)
Routing:
- added copper zone on F.Cu, net signal
Other:
- board text added: "NV diamond 2026 Physics 108 ML"
Changed lines of the file:
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@@
 	(net 0 "")
 	(net 1 "gnd")
+	(net 2 "signal")
+	(footprint "custom:open-mask"
+		(layer "F.Cu")
+		(at 75.28 100.25)
+		(property "Reference" "REF**"
+			(at 0 -0.5 0)
+			(unlocked yes)
+			(layer "F.SilkS")
+			(hide yes)
+			(effects
+				(font
+					(size 1 1)
+					(thickness 0.1)
+				)
+			)
+		)
+		(property "Value" "signal"
+			(at -2.415 0 0)
+			(unlocked yes)
+			(layer "F.Fab")
+			(effects
+				(font
+					(size 1 1)
+					(thickness 0.15)
+				)
+			)
+		)
+		(property "Datasheet" ""
+			(at 0 0 0)
+			(unlocked yes)
+			(layer "F.Fab")
+			(hide yes)
+			(effects
+				(font
+					(size 1 1)
+					(thickness 0.15)
+				)
+			)
+		)
+		(property "Description" ""
+			(at 0 0 0)
+			(unlocked yes)
+			(layer "F.Fab")
+			(hide yes)
+			(effects
+				(font
+					(size 1 1)
+					(thickness 0.15)
+				)
+			)
+		)
+		(attr smd)
+		(fp_poly
+			(pts
+				(xy 0 -1.077444) (xy -5.08 -1.4) (xy -5.08 1.4) (xy 0 1.077444)
+			)
+			(stroke
+				(width 0)
+				(type solid)
+			)
+			(fill yes)
+			(layer "F.Mask")
+		)
+		(embedded_fonts no)
+	)
 	(footprint "clipboard:33e20c2f-486e-44d1-b761-1e7e435959c7"
 		(layer "F.Cu")
@@
 		)
 		(pad "1" smd rect
-			(at 0 -8.76)
+			(at 0 -8.9825)
 			(size 5.08 2.42)
 			(layers "B.Cu" "B.Mask" "B.Paste")
@@
 		)
 		(pad "1" smd rect
-			(at 0 0)
+			(at 0 -0.2175)
 			(size 5.08 2.42)
 			(layers "B.Cu" "B.Mask" "B.Paste")
@@
 		)
 		(embedded_fonts no)
-	)
-	(gr_circle
-		(center 100 100)
-		(end 108 100)
-		(stroke
-			(width 0.01)
-			(type solid)
-		)
-		(fill no)
-		(locked yes)
-		(layer "F.Cu")
-	)
-	(gr_line
-		(start 92.05 100.1)
-		(end 92.05 100.4)
-		(stroke
-			(width 0.01)
-			(type solid)
-		)
-		(layer "F.Cu")
-	)
-	(gr_rect
-		(start 91.99 99.9)
-		(end 102.99 100.1)
-		(stroke
-			(width 0.01)
-			(type solid)
-		)
-		(fill no)
-		(locked yes)
-		(layer "F.Cu")
-	)
-	(gr_line
-		(start 70 98.85)
-		(end 70 101.65)
-		(stroke
-			(width 0.01)
-			(type solid)
-		)
-		(layer "F.Cu")
-	)
-	(gr_line
-		(start 92.05 100.1)
-		(end 70 98.85)
-		(stroke
-			(width 0.01)
-			(type solid)
-		)
-		(layer "F.Cu")
-	)
-	(gr_circle
-		(center 103 100)
-		(end 103.5 100)
-		(stroke
-			(width 0.01)
-			(type solid)
-		)
-		(fill no)
-		(locked yes)
-		(layer "F.Cu")
-	)
-	(gr_line
-		(start 70 101.65)
-		(end 92.05 100.4)
-		(stroke
-			(width 0.01)
-			(type solid)
-		)
-		(layer "F.Cu")
 	)
 	(gr_rect
@@
 		(layer "Edge.Cuts")
 	)
-	(zone
+	(gr_text "NV diamond 2026\nPhysics 108\nML"
+		(at 106.1 92.9 0)
+		(layer "F.SilkS")
+		(effects
+			(font
+				(size 1 1)
+				(thickness 0.1)
+			)
+			(justify left bottom)
+		)
+	)
+	(zone
+		(net 2)
+		(net_name "signal")
+		(layer "F.Cu")
+		(hatch edge 0.5)
+		(connect_pads
+			(clearance 0)
+		)
+		(min_thickness 0.025)
+		(filled_areas_thickness no)
+		(fill yes
+			(thermal_gap 0.5)
+			(thermal_bridge_width 0.5)
+			(island_removal_mode 1)
+			(island_area_min 10)
+		)
+		(polygon
+			(pts
+				(xy 70 98.85) (xy 92.05 100.1) (xy 92.05 100.4) (xy 70 101.65)
+			)
+		)
+	)
+	(zone
+		(net 2)
+		(net_name "signal")
+		(layer "F.Cu")
+		(hatch edge 0.5)
+		(connect_pads
+			(clearance 0)
+		)
+		(min_thickness 0.025)
+		(filled_areas_thickness no)
+		(fill yes
+			(thermal_gap 0.5)
+			(thermal_bridge_width 0.5)
+			(island_removal_mode 1)
+			(island_area_min 10)
+		)
+		(polygon
+			(pts
+				(arc
+					(start 92 100)
+					(mid 108 100)
+					(end 92 100)
+				)
+			)
+		)
+	)
+	(zone
+		(net 0)
+		(net_name "")
+		(layer "F.Cu")
+		(hatch edge 0.5)
+		(connect_pads
+			(clearance 0)
+		)
+		(min_thickness 0.025)
+		(filled_areas_thickness no)
+		(keepout
+			(tracks not_allowed)
+			(vias not_allowed)
+			(pads not_allowed)
+			(copperpour not_allowed)
+			(footprints allowed)
+		)
+		(placement
+			(enabled no)
+			(sheetname "")
+		)
+		(fill
+			(thermal_gap 0.5)
+			(thermal_bridge_width 0.5)
+			(island_removal_mode 1)
+			(island_area_min 10)
+		)
+		(polygon
+			(pts
+				(arc
+					(start 102.5 100)
+					(mid 103.5 100)
+					(end 102.5 100)
+				)
+			)
+		)
+	)
+	(zone
+		(net 0)
+		(net_name "")
+		(layer "F.Cu")
+		(hatch edge 0.5)
+		(connect_pads
+			(clearance 0)
+		)
+		(min_thickness 0.025)
+		(filled_areas_thickness no)
+		(keepout
+			(tracks not_allowed)
+			(vias not_allowed)
+			(pads not_allowed)
+			(copperpour not_allowed)
+			(footprints allowed)
+		)
+		(placement
+			(enabled no)
+			(sheetname "")
+		)
+		(fill
+			(thermal_gap 0.5)
+			(thermal_bridge_width 0.5)
+			(island_removal_mode 1)
+			(island_area_min 10)
+		)
+		(polygon
+			(pts
+				(xy 91.99 99.9) (xy 102.99 99.9) (xy 102.99 100.1) (xy 91.99 100.1)
+			)
+		)
+	)
+	(zone
